Commit message: stuff

File: urdf/dropbear/urdf/dropbear.urdf (robot description, URDF)
Before this commit: robot biped_robot, 12 links, 8 joints
Links:
- removed link left_hip_pitch_knee_front_bracket
- removed link left_hip_pitch_knee_rear_bracket
- removed link left_knee_secondary_hanger
- removed link right_knee_secondary_hanger
- added link left_ankle; visual mesh filename=../meshes/ankle.stl scale=0.05 0.05 0.05
- added link left_foot; visual mesh filename=../meshes/foot.stl scale=0.05 0.05 0.05
- added link left_hip_pitch_knee_motors; visual mesh filename=../meshes/leftHipPitchKneeMotors.stl scale=0.05 0.05 0.05
- added link left_hip_roll_motor; visual mesh filename=../meshes/leftHipRollMotor.stl scale=0.05 0.05 0.05
- added link right_ankle; visual mesh filename=../meshes/ankle.stl scale=0.05 0.05 0.05
- added link right_foot; visual mesh filename=../meshes/foot.stl scale=0.05 0.05 0.05
- added link right_hip_pitch_knee_motors; visual mesh filename=../meshes/rightHipPitchKneeMotors.stl scale=0.05 0.05 0.05
- added link right_hip_roll_motor; visual mesh filename=../meshes/rightHipRollMotor.stl scale=0.05 0.05 0.05
- link hips: geometry visual mesh filename=../meshes/hipRollAssembly.stl scale=0.05 0.05 0.05
- link left_calf: geometry visual mesh filename=../meshes/leftCalf.stl scale=0.05 0.05 0.05
- link left_knee_primary_hanger: geometry visual mesh filename=../meshes/kneePrimaryHangar.stl scale=0.05 0.05 0.05
- link right_calf: geometry visual mesh filename=../meshes/rightCalf.stl scale=0.05 0.05 0.05
- link right_hip_pitch_knee_front_bracket: geometry visual mesh filename=../meshes/rightHipPitchKneeFrontBracket.stl scale=0.05 0.05 0.05
- link right_hip_pitch_knee_rear_bracket: geometry visual mesh filename=../meshes/rightHipPitchKneeRearBracket.stl scale=0.05 0.05 0.05
- link right_knee_primary_hanger: geometry visual mesh filename=../meshes/kneePrimaryHangar.stl scale=0.05 0.05 0.05
- link torso: geometry visual mesh filename=../meshes/torso.stl scale=0.05 0.05 0.05
Joints:
- removed joint left_calf_to_primary_hanger
- removed joint left_hip_joint
- removed joint left_knee_front_to_primary_hanger
- removed joint left_knee_rear_to_primary_hanger
- removed joint right_calf_to_primary_hanger
- removed joint right_hip_joint
- removed joint right_knee_front_to_primary_hanger
- removed joint right_knee_rear_to_primary_hanger
- added joint left_ankle_joint: type revolute, parent left_calf, child left_ankle, origin xyz=0 0 -0.05 rpy=0 0 0, axis 1 0 0, limit lower=-0.785 upper=0.785 effort=0 velocity=0
- added joint left_foot_joint: type revolute, parent left_ankle, child left_foot, origin xyz=0 0 -0.05 rpy=0 0 0, axis 1 0 0, limit lower=-0.785 upper=0.785 effort=0 velocity=0
- added joint left_hip_pitch_joint: type revolute, parent left_hip_roll_motor, child left_hip_pitch_knee_motors, origin xyz=0 0 -0.05 rpy=0 0 0, axis 0 1 0, limit lower=-1.57 upper=1.57 effort=0 velocity=0
- added joint left_hip_roll_joint: type revolute, parent hips, child left_hip_roll_motor, origin xyz=0 0.1 0 rpy=0 0 0, axis 0 1 0, limit lower=-0.785 upper=0.785 effort=0 velocity=0
- added joint left_knee_primary_hanger_joint: type revolute, parent left_hip_pitch_knee_motors, child left_knee_primary_hanger, origin xyz=0 0 -0.1 rpy=0 0 0, axis 0 0 1, limit lower=-2.356 upper=0 effort=0 velocity=0
- added joint left_knee_to_calf_joint: type revolute, parent left_knee_primary_hanger, child left_calf, origin xyz=0 0 -0.2 rpy=0 0 0, axis 0 1 0, limit lower=-0.523 upper=0.523 effort=0 velocity=0
- added joint right_ankle_joint: type revolute, parent right_calf, child right_ankle, origin xyz=0 -10 -0.05 rpy=0 0 0, axis 1 0 0, limit lower=-0.785 upper=0.785 effort=0 velocity=0
- added joint right_foot_joint: type revolute, parent right_ankle, child right_foot, origin xyz=0 0 -0.05 rpy=0 0 0, axis 1 0 0, limit lower=-0.785 upper=0.785 effort=0 velocity=0
- added joint right_hip_pitch_joint: type revolute, parent right_hip_roll_motor, child right_hip_pitch_knee_motors, origin xyz=0 0 -0.05 rpy=0 0 0, axis 0 1 0, limit lower=-1.57 upper=1.57 effort=0 velocity=0
- added joint right_hip_pitch_to_front_bracket_joint: type revolute, parent right_hip_pitch_knee_motors, child right_hip_pitch_knee_front_bracket, origin xyz=0 0 -0.1 rpy=0 0 0, axis 1 0 0, limit lower=-1.57 upper=1.57 effort=0 velocity=0
- added joint right_hip_roll_joint: type revolute, parent hips, child right_hip_roll_motor, origin xyz=0 0 0 rpy=0 0 0, axis 0 1 0, limit lower=-0.785 upper=0.785 effort=0 velocity=0
- added joint right_knee_primary_hanger_joint: type revolute, parent right_hip_pitch_knee_front_bracket, child right_knee_primary_hanger, origin xyz=0 0 -0.1 rpy=0 0 0, axis 0 0 1, limit lower=-2.356 upper=0 effort=0 velocity=0
- added joint right_knee_to_calf_joint: type revolute, parent right_knee_primary_hanger, child right_calf, origin xyz=0 0 -0.2 rpy=0 0 0, axis 0 1 0, limit lower=-0.523 upper=0.523 effort=0 velocity=0
- added joint torso_to_hips_joint: type fixed, parent torso, child hips, origin xyz=-5 -26 2.25 rpy=0 0 0

Commit message: update urdf meshes live!

File: urdf/dropbear/urdf/dropbear.urdf (robot description, URDF)
Before this commit: robot biped_robot, 16 links, 14 joints
Joints:
- joint torso_to_hips_joint: origin xyz=-5 -26 2.25 rpy=0 0 0 -> xyz=-10 -26 2.25 rpy=0 0 0

Commit message: interface

File: urdf/dropbear/urdf/dropbear.urdf (robot description, URDF)
Before this commit: robot biped_robot, 16 links, 14 joints
Joints:
- joint torso_to_hips_joint: origin xyz=-10 -26 2.25 rpy=0 0 0 -> xyz=-2 -26 2.25 rpy=0 0 0

Commit message: conditional decimal places

File: urdf/dropbear/urdf/dropbear.urdf (robot description, URDF)
Before this commit: robot biped_robot, 16 links, 14 joints
Joints:
- joint right_hip_pitch_joint: axis 0 1 0 -> 0.00 1.00 0.00; limit lower=-1.57 upper=1.57 effort=0 velocity=0 -> lower=-89.95 upper=89.95 effort=0 velocity=0; origin xyz=0 0 -0.05 rpy=0 0 0 -> xyz=0 0 10.05 rpy=0.00 0.00 0.00
- joint right_hip_pitch_to_front_bracket_joint: axis 1 0 0 -> 0.00 1.00 0.00; limit lower=-1.57 upper=1.57 effort=0 velocity=0 -> lower=-89.95 upper=89.95 effort=0 velocity=0; origin xyz=0 0 -0.1 rpy=0 0 0 -> xyz=0 0 -0.05 rpy=0.00 0.00 0.00
- joint right_knee_to_calf_joint: axis 0 1 0 -> 0.00 0.00 1.00; limit lower=-0.523 upper=0.523 effort=0 velocity=0 -> lower=-29.97 upper=29.97 effort=0 velocity=0; origin xyz=0 0 -0.2 rpy=0 0 0 -> xyz=0 -29 10 rpy=0.00 0.00 5.00

Commit message: fies to urdf update joint labeling

File: urdf/dropbear/urdf/dropbear.urdf (robot description, URDF)
Before this commit: robot biped_robot, 16 links, 14 joints
Joints:
- joint left_foot_joint: axis 1 0 0 -> 0 1.0 0; limit lower=-0.785 upper=0.785 effort=0 velocity=0 -> lower=-295451.4 upper=295451.4 effort=0 velocity=0; origin xyz=0 0 -0.05 rpy=0 0 0 -> xyz=0 -0 -10.05 rpy=0 0 0
- joint left_hip_pitch_joint: axis 0 1 0 -> 0 1.0 0; limit lower=-1.57 upper=1.57 effort=0 velocity=0 -> lower=-90.0 upper=90.0 effort=0 velocity=0; origin xyz=0 0 -0.05 rpy=0 0 0 -> xyz=0 0 -10.05 rpy=0 0 0
- joint left_knee_to_calf_joint: axis 0 1 0 -> 0 1.0 0; limit lower=-0.523 upper=0.523 effort=0 velocity=0 -> lower=-90.0 upper=90.0 effort=0 velocity=0; origin xyz=0 0 -0.2 rpy=0 0 0 -> xyz=0 0 10.05 rpy=0 0 0
- joint right_hip_pitch_joint: axis 0.00 1.00 0.00 -> 0 1.0 0; limit lower=-89.95 upper=89.95 effort=0 velocity=0 -> lower=-295451.4 upper=295451.4 effort=0 velocity=0; origin xyz=0 0 10.05 rpy=0.00 0.00 0.00 -> xyz=0 0 10.05 rpy=0 0 0
- joint right_hip_pitch_to_front_bracket_joint: axis 0.00 1.00 0.00 -> 0 1.0 0; limit lower=-89.95 upper=89.95 effort=0 velocity=0 -> lower=-295451.4 upper=295451.4 effort=0 velocity=0; origin xyz=0 0 -0.05 rpy=0.00 0.00 0.00 -> xyz=5 -2.5 -9 rpy=0 0 0
- joint right_knee_primary_hanger_joint: axis 0 0 1 -> 0 1.0 0; limit lower=-2.356 upper=0 effort=0 velocity=0 -> lower=-16928118.3 upper=16928118.3 effort=0 velocity=0; origin xyz=0 0 -0.1 rpy=0 0 0 -> xyz=-2 -12 12 rpy=0 0 0
- joint right_knee_to_calf_joint: axis 0.00 0.00 1.00 -> 0 1.0 0; limit lower=-29.97 upper=29.97 effort=0 velocity=0 -> lower=-90.0 upper=90.0 effort=0 velocity=0; origin xyz=0 -29 10 rpy=0.00 0.00 5.00 -> xyz=0 0 -10.05 rpy=0 0 0

Commit message: minor fixes

File: urdf/dropbear/urdf/dropbear.urdf (robot description, URDF)
Before this commit: robot biped_robot, 16 links, 14 joints
Joints:
- joint left_hip_roll_joint: axis 0 1 0 -> 0 1.0 0; limit lower=-0.785 upper=0.785 effort=0 velocity=0 -> lower=-2578.3 upper=2578.3 effort=0 velocity=0; origin xyz=0 0.1 0 rpy=0 0 0 -> xyz=0 0 -4 rpy=0 0 0
- joint right_ankle_joint: axis 1 0 0 -> 0 0 1.0; limit lower=-0.785 upper=0.785 effort=0 velocity=0 -> lower=-45.0 upper=45.0 effort=0 velocity=0; origin xyz=0 -10 -0.05 rpy=0 0 0 -> xyz=0 -14 -0.05 rpy=0 0 0
- joint right_foot_joint: axis 1 0 0 -> 1.0 0 0; limit lower=-0.785 upper=0.785 effort=0 velocity=0 -> lower=-45.0 upper=45.0 effort=0 velocity=0
- joint right_hip_pitch_joint: axis 0 1.0 0 -> 0 0 1.0; limit lower=-295451.4 upper=295451.4 effort=0 velocity=0 -> lower=-969909733.7 upper=969909733.7 effort=0 velocity=0; origin xyz=0 0 10.05 rpy=0 0 0 -> xyz=0 -7 2 rpy=0 0 0
- joint right_hip_pitch_to_front_bracket_joint: limit lower=-295451.4 upper=295451.4 effort=0 velocity=0 -> lower=-16928118.3 upper=16928118.3 effort=0 velocity=0; origin xyz=5 -2.5 -9 rpy=0 0 0 -> xyz=10 3.5 -9 rpy=0 0 0
- joint right_hip_roll_joint: axis 0 1 0 -> 0 1.0 0; limit lower=-0.785 upper=0.785 effort=0 velocity=0 -> lower=-45.0 upper=45.0 effort=0 velocity=0; origin xyz=0 0 0 rpy=0 0 0 -> xyz=0 0 4 rpy=0 0 0
- joint right_knee_primary_hanger_joint: axis 0 1.0 0 -> 0 0 1.0; limit lower=-16928118.3 upper=16928118.3 effort=0 velocity=0 -> lower=-45 upper=45 effort=0 velocity=0; origin xyz=-2 -12 12 rpy=0 0 0 -> xyz=-5.5 -17 13 rpy=0 0 0
- joint right_knee_to_calf_joint: limit lower=-90.0 upper=90.0 effort=0 velocity=0 -> lower=-5156.6 upper=5156.6 effort=0 velocity=0; origin xyz=0 0 -10.05 rpy=0 0 0 -> xyz=0 -13.5 1.5 rpy=0 0 0
- joint torso_to_hips_joint: axis (none) -> 0 1.0 0; limit (none) -> lower=-45.0 upper=45.0; origin xyz=-2 -26 2.25 rpy=0 0 0 -> xyz=-4.5 -26 2.25 rpy=0 0 0

Commit message: corrected parsing of child index dependant on kinematics chain position

File: urdf/dropbear/urdf/dropbear.urdf (robot description, URDF)
Before this commit: robot biped_robot, 16 links, 14 joints
Joints:
- joint right_hip_pitch_to_front_bracket_joint: axis 0 1.0 0 -> 0 0 1; limit lower=-16928118.3 upper=16928118.3 effort=0 velocity=0 -> lower=-969909733.7 upper=969909733.7 effort=0 velocity=0

Commit message: further fixes for parsing and writing link states to urdf

File: urdf/dropbear/urdf/dropbear.urdf (robot description, URDF)
Before this commit: robot biped_robot, 16 links, 14 joints
Joints:
- joint right_hip_pitch_to_front_bracket_joint: axis 0 0 1 -> 0 0 1.0; limit lower=-969909733.7 upper=969909733.7 effort=0 velocity=0 -> lower=-55571734249.7 upper=55571734249.7 effort=0 velocity=0; origin xyz=10 3.5 -9 rpy=0 0 0 -> xyz=7 3.5 0 rpy=0 0 0
- joint right_knee_primary_hanger_joint: limit lower=-45 upper=45 effort=0 velocity=0 -> lower=-147725.7 upper=147725.7 effort=0 velocity=0; origin xyz=-5.5 -17 13 rpy=0 0 0 -> xyz=-5.5 -17 0 rpy=0 0 0

Commit message: conversion of deg from joint rpy input box input to radian, then to quaternion for model, and back again when joint selected

File: urdf/dropbear/urdf/dropbear.urdf (robot description, URDF)
Before this commit: robot biped_robot, 16 links, 14 joints
Joints:
- joint right_ankle_joint: axis 0 0 1.0 -> 1.0 0 0; limit lower=-45.0 upper=45.0 effort=0 velocity=0 -> lower=-90.0 upper=90.0 effort=0 velocity=0; origin xyz=0 -14 -0.05 rpy=0 0 0 -> xyz=2.2 -21.5 3 rpy=-10.0 90.0 0
- joint right_foot_joint: limit lower=-45.0 upper=45.0 effort=0 velocity=0 -> lower=-90.0 upper=90.0 effort=0 velocity=0; origin xyz=0 0 -0.05 rpy=0 0 0 -> xyz=0 -2 1.2 rpy=0 -90.0 0
- joint right_hip_pitch_joint: limit lower=-969909733.7 upper=969909733.7 effort=0 velocity=0 -> lower=-90.0 upper=90.0 effort=0 velocity=0; origin xyz=0 -7 2 rpy=0 0 0 -> xyz=0 -5 2 rpy=-0.1745329 0 0
- joint right_hip_pitch_to_front_bracket_joint: limit lower=-55571734249.7 upper=55571734249.7 effort=0 velocity=0 -> lower=-3184025832730.4 upper=3184025832730.4 effort=0 velocity=0; origin xyz=7 3.5 0 rpy=0 0 0 -> xyz=2.48 -0.8 3.6 rpy=0 0 0
- joint right_hip_roll_joint: axis 0 1.0 0 -> 1.0 0 0; limit lower=-45.0 upper=45.0 effort=0 velocity=0 -> lower=-2578.3 upper=2578.3 effort=0 velocity=0; origin xyz=0 0 4 rpy=0 0 0 -> xyz=1.1 0 3 rpy=0 0 0
- joint right_knee_primary_hanger_joint: limit lower=-147725.7 upper=147725.7 effort=0 velocity=0 -> lower=-8464059.1 upper=8464059.1 effort=0 velocity=0; origin xyz=-5.5 -17 0 rpy=0 0 0 -> xyz=-2 -17 -0.75 rpy=0 0 0
- joint right_knee_to_calf_joint: axis 0 1.0 0 -> 0 0 1.0; limit lower=-5156.6 upper=5156.6 effort=0 velocity=0 -> lower=-16928118.3 upper=16928118.3 effort=0 velocity=0; origin xyz=0 -13.5 1.5 rpy=0 0 0 -> xyz=0 -3 1.5 rpy=0 0 0

Commit message: interface styling

File: urdf/dropbear/urdf/dropbear.urdf (robot description, URDF)
Before this commit: robot biped_robot, 16 links, 14 joints
Joints:
- joint right_ankle_joint: limit lower=-90.0 upper=90.0 effort=0 velocity=0 -> lower=-89.9996482083396 upper=89.9996482083396 effort=0 velocity=0; origin xyz=2.2 -21.5 3 rpy=-10.0 90.0 0 -> xyz=2.2 -21.5 3 rpy=0 1.5707963267948966 0
- joint right_foot_joint: limit lower=-90.0 upper=90.0 effort=0 velocity=0 -> lower=-89.9996482083396 upper=89.9996482083396 effort=0 velocity=0; origin xyz=0 -2 1.2 rpy=0 -90.0 0 -> xyz=0 -2 1.2 rpy=0 -1.5707963267948966 0
- joint right_hip_pitch_joint: limit lower=-90.0 upper=90.0 effort=0 velocity=0 -> lower=-89.9996482083396 upper=89.9996482083396 effort=0 velocity=0; origin xyz=0 -5 2 rpy=-0.1745329 0 0 -> xyz=0 -5 2 rpy=0.17453292519943295 0 0

Commit message: corrected all joint limits in dropbear URDF

File: urdf/dropbear/urdf/dropbear.urdf (robot description, URDF)
Before this commit: robot biped_robot, 16 links, 14 joints
Joints:
- joint left_ankle_joint: limit lower=-0.785 upper=0.785 effort=0 velocity=0 -> lower=-6.28319 upper=6.28319 effort=0 velocity=0
- joint left_foot_joint: limit lower=-295451.4 upper=295451.4 effort=0 velocity=0 -> lower=-6.28319 upper=6.28319 effort=0 velocity=0
- joint left_hip_pitch_joint: limit lower=-90.0 upper=90.0 effort=0 velocity=0 -> lower=-6.28319 upper=6.28319 effort=0 velocity=0
- joint left_hip_roll_joint: limit lower=-2578.3 upper=2578.3 effort=0 velocity=0 -> lower=-6.28319 upper=6.28319 effort=0 velocity=0
- joint left_knee_primary_hanger_joint: limit lower=-2.356 upper=0 effort=0 velocity=0 -> lower=-6.28319 upper=6.28319 effort=0 velocity=0
- joint left_knee_to_calf_joint: limit lower=-90.0 upper=90.0 effort=0 velocity=0 -> lower=-6.28319 upper=6.28319 effort=0 velocity=0
- joint right_ankle_joint: limit lower=-89.9996482083396 upper=89.9996482083396 effort=0 velocity=0 -> lower=-6.28319 upper=6.28319 effort=0 velocity=0
- joint right_foot_joint: limit lower=-89.9996482083396 upper=89.9996482083396 effort=0 velocity=0 -> lower=-6.28319 upper=6.28319 effort=0 velocity=0
- joint right_hip_pitch_joint: limit lower=-89.9996482083396 upper=89.9996482083396 effort=0 velocity=0 -> lower=-6.28319 upper=6.28319 effort=0 velocity=0
- joint right_hip_pitch_to_front_bracket_joint: limit lower=-3184025832730.4 upper=3184025832730.4 effort=0 velocity=0 -> lower=-6.28319 upper=6.28319 effort=0 velocity=0
- joint right_hip_roll_joint: limit lower=-2578.3 upper=2578.3 effort=0 velocity=0 -> lower=-6.28319 upper=6.28319 effort=0 velocity=0
- joint right_knee_primary_hanger_joint: limit lower=-8464059.1 upper=8464059.1 effort=0 velocity=0 -> lower=-6.28319 upper=6.28319 effort=0 velocity=0
- joint right_knee_to_calf_joint: limit lower=-16928118.3 upper=16928118.3 effort=0 velocity=0 -> lower=-6.28319 upper=6.28319 effort=0 velocity=0

Commit message: corrected urdf

File: urdf/dropbear/urdf/dropbear.urdf (robot description, URDF)
Before this commit: robot biped_robot, 16 links, 14 joints
Links:
- removed link hips
- removed link left_ankle
- removed link left_calf
- removed link left_foot
- removed link left_hip_pitch_knee_motors
- removed link left_hip_roll_motor
- removed link left_knee_primary_hanger
- removed link right_ankle
- removed link right_calf
- removed link right_foot
- removed link right_hip_pitch_knee_front_bracket
- removed link right_hip_pitch_knee_motors
- removed link right_hip_pitch_knee_rear_bracket
- removed link right_hip_roll_motor
- removed link right_knee_primary_hanger
- added link ankle; visual mesh filename=../meshes/ankle.stl scale=0.05 0.05 0.05
- added link foot; visual mesh filename=../meshes/foot.stl scale=0.05 0.05 0.05
- added link hipRollAssembly; visual mesh filename=../meshes/hipRollAssembly.stl scale=0.05 0.05 0.05
- added link hipYawBracket; visual mesh filename=../meshes/hipYawBracket.stl scale=0.05 0.05 0.05
- added link rightCalf; visual mesh filename=../meshes/rightCalf.stl scale=0.05 0.05 0.05
- added link rightHipPitchKneeFrontBracket; visual mesh filename=../meshes/rightHipPitchKneeFrontBracket.stl scale=0.05 0.05 0.05
- added link rightHipPitchKneeMotors; visual mesh filename=../meshes/rightHipPitchKneeMotors.stl scale=0.05 0.05 0.05
- added link rightHipPitchKneeRearBracket; visual mesh filename=../meshes/rightHipPitchKneeRearBracket.stl scale=0.05 0.05 0.05
- added link rightHipRollMotor; visual mesh filename=../meshes/rightHipRollMotor.stl scale=0.05 0.05 0.05
- added link rightKneePrimaryHangar; visual mesh filename=../meshes/kneePrimaryHangar.stl scale=0.05 0.05 0.05
- added link rightKneeSecondaryHangar; visual mesh filename=../meshes/kneeSecondaryHangar.stl scale=0.05 0.05 0.05
Joints:
- removed joint left_ankle_joint
- removed joint left_foot_joint
- removed joint left_hip_pitch_joint
- removed joint left_hip_roll_joint
- removed joint left_knee_primary_hanger_joint
- removed joint left_knee_to_calf_joint
- removed joint right_ankle_joint
- removed joint right_foot_joint
- removed joint right_hip_pitch_joint
- removed joint right_hip_pitch_to_front_bracket_joint
- removed joint right_hip_roll_joint
- removed joint right_knee_primary_hanger_joint
- removed joint right_knee_to_calf_joint
- added joint ankle_to_foot: type revolute, parent ankle, child foot, origin xyz=0 -2 1.2 rpy=0 -1.5707963267948966 0, axis 1.0 0 0, limit lower=-6.283185307179586 upper=6.283185307179586 effort=0 velocity=0
- added joint hipRollAssembly_to_rightHipRollMotor: type revolute, parent hipRollAssembly, child rightHipRollMotor, origin xyz=1.1 0 3 rpy=0.17453292519943295 0 0, axis 1.0 0 0, limit lower=-6.283185307179586 upper=6.283185307179586 effort=0 velocity=0
- added joint hipYawBracket_to_rightHipPitchKneeMotors: type revolute, parent hipYawBracket, child rightHipPitchKneeMotors, origin xyz=0 -3 3 rpy=0 0 -0.06981317007977318, axis 0 0 1.0, limit lower=-6.283185307179586 upper=6.283185307179586 effort=0 velocity=0
- added joint rightCalf_to_ankle: type revolute, parent rightCalf, child ankle, origin xyz=3.5 -21.5 2 rpy=-0.17453292519943295 1.5707963267948966 0, axis 1.0 0 0, limit lower=-6.283185307179586 upper=6.283185307179586 effort=0 velocity=0
- added joint rightHipPitchKneeFrontBracket_to_rightKneePrimaryHangar: type revolute, parent rightHipPitchKneeFrontBracket, child rightKneePrimaryHangar, origin xyz=-0.1 -16 -0.75 rpy=0 0 0, axis 0 0 1.0, limit lower=-6.283185307179586 upper=6.283185307179586 effort=0 velocity=0
- added joint rightHipPitchKneeFrontBracket_to_rightKneeSecondaryHangar: type revolute, parent rightHipPitchKneeFrontBracket, child rightKneeSecondaryHangar, origin xyz=-3.2 -16.7 -0.8 rpy=0 0 0.17453292519943295, axis 0 0 1.0, limit lower=-6.283185307179586 upper=6.283185307179586 effort=0 velocity=0
- added joint rightHipPitchKneeMotors_to_rightHipPitchKneeFrontBracket: type revolute, parent rightHipPitchKneeMotors, child rightHipPitchKneeFrontBracket, origin xyz=2.48 -0.8 3.6 rpy=0 0 0, axis 0 0 1.0, limit lower=-6.283185307179586 upper=6.283185307179586 effort=0 velocity=0
- added joint rightHipPitchKneeMotors_to_rightHipPitchKneeRearBracket: type revolute, parent rightHipPitchKneeMotors, child rightHipPitchKneeRearBracket, origin xyz=-4 -5 3 rpy=0 0 0, axis 0 0 1.0, limit lower=-6.283185307179586 upper=6.283185307179586 effort=0 velocity=0
- added joint rightHipRollMotor_to_hipYawBracket: type revolute, parent rightHipRollMotor, child hipYawBracket, origin xyz=1 -2 0 rpy=0 0 0, axis 0 1.0 0, limit lower=-6.283185307179586 upper=6.283185307179586 effort=0 velocity=0
- added joint rightKneePrimaryHangar_to_rightCalf: type revolute, parent rightKneePrimaryHangar, child rightCalf, origin xyz=-3.65 -5 1.5 rpy=0 0 0, axis 0 0 1.0, limit lower=-6.283185307179586 upper=6.283185307179586 effort=0 velocity=0
- joint torso_to_hips_joint: axis 0 1.0 0 -> 0 1 0; child hips -> hipRollAssembly; origin xyz=-4.5 -26 2.25 rpy=0 0 0 -> xyz=0 0 0 rpy=0 0 0

Commit message: correctly access urdf content from uploaded urdf files by  apply and edit urdf functions

File: urdf/dropbear/urdf/dropbear.urdf (robot description, URDF)
Before this commit: robot biped_robot, 12 links, 11 joints
Links:
- link ankle: geometry visual mesh filename=../meshes/ankle.stl scale=0.01 0.01 0.01
- link foot: geometry visual mesh filename=../meshes/foot.stl scale=0.01 0.01 0.01
- link hipRollAssembly: geometry visual mesh filename=../meshes/hipRollAssembly.stl scale=0.01 0.01 0.01
- link hipYawBracket: geometry visual mesh filename=../meshes/hipYawBracket.stl scale=0.01 0.01 0.01
- link rightCalf: geometry visual mesh filename=../meshes/rightCalf.stl scale=0.01 0.01 0.01
- link rightHipPitchKneeFrontBracket: geometry visual mesh filename=../meshes/rightHipPitchKneeFrontBracket.stl scale=0.01 0.01 0.01
- link rightHipPitchKneeMotors: geometry visual mesh filename=../meshes/rightHipPitchKneeMotors.stl scale=0.01 0.01 0.01
- link rightHipPitchKneeRearBracket: geometry visual mesh filename=../meshes/rightHipPitchKneeRearBracket.stl scale=0.01 0.01 0.01
- link rightHipRollMotor: geometry visual mesh filename=../meshes/rightHipRollMotor.stl scale=0.01 0.01 0.01
- link rightKneePrimaryHangar: geometry visual mesh filename=../meshes/kneePrimaryHangar.stl scale=0.01 0.01 0.01
- link rightKneeSecondaryHangar: geometry visual mesh filename=../meshes/kneeSecondaryHangar.stl scale=0.01 0.01 0.01
- link torso: geometry visual mesh filename=../meshes/torso.stl scale=0.01 0.01 0.01
