Commit message: debugging

File: urdf/dropbear/urdf/dropbear.urdf (robot description, URDF)
Before this commit: robot biped_robot, 12 links, 11 joints
Links:
- link ankle: geometry visual mesh filename=../meshes/ankle.stl scale=0.05 0.05 0.05
- link foot: geometry visual mesh filename=../meshes/foot.stl scale=0.05 0.05 0.05
- link hipRollAssembly: geometry visual mesh filename=../meshes/hipRollAssembly.stl scale=0.05 0.05 0.05
- link hipYawBracket: geometry visual mesh filename=../meshes/hipYawBracket.stl scale=0.05 0.05 0.05
- link rightCalf: geometry visual mesh filename=../meshes/rightCalf.stl scale=0.05 0.05 0.05
- link rightHipPitchKneeFrontBracket: geometry visual mesh filename=../meshes/rightHipPitchKneeFrontBracket.stl scale=0.05 0.05 0.05
- link rightHipPitchKneeMotors: geometry visual mesh filename=../meshes/rightHipPitchKneeMotors.stl scale=0.05 0.05 0.05
- link rightHipPitchKneeRearBracket: geometry visual mesh filename=../meshes/rightHipPitchKneeRearBracket.stl scale=0.05 0.05 0.05
- link rightHipRollMotor: geometry visual mesh filename=../meshes/rightHipRollMotor.stl scale=0.05 0.05 0.05
- link rightKneePrimaryHangar: geometry visual mesh filename=../meshes/kneePrimaryHangar.stl scale=0.05 0.05 0.05
- link rightKneeSecondaryHangar: geometry visual mesh filename=../meshes/kneeSecondaryHangar.stl scale=0.05 0.05 0.05
- link torso: geometry visual mesh filename=../meshes/torso.stl scale=0.05 0.05 0.05

Commit message: stable

File: urdf/dropbear/urdf/dropbear.urdf (robot description, URDF)
Before this commit: robot biped_robot, 12 links, 11 joints
Joints:
- joint rightHipPitchKneeMotors_to_rightHipPitchKneeRearBracket: mimic (none) -> joint=rightHipPitchKneeMotors_to_rightHipPitchKneeFrontBracket multiplier=0.9 offset=0; type revolute -> mimic

Commit message: mimic joint functionality

File: urdf/dropbear/urdf/dropbear.urdf (robot description, URDF)
Before this commit: robot biped_robot, 12 links, 11 joints
Joints:
- joint rightHipPitchKneeMotors_to_rightHipPitchKneeRearBracket: mimic joint=rightHipPitchKneeMotors_to_rightHipPitchKneeFrontBracket multiplier=0.9 offset=0 -> joint=rightHipPitchKneeMotors_to_rightHipPitchKneeFrontBracket multiplier=0.5 offset=0

Commit message: updated urdf

File: urdf/dropbear/urdf/dropbear.urdf (robot description, URDF)
Before this commit: robot biped_robot, 12 links, 11 joints
Joints:
- joint rightHipPitchKneeFrontBracket_to_rightKneePrimaryHangar: mimic (none) -> joint=rightHipPitchKneeMotors_to_rightHipPitchKneeFrontBracket multiplier=-1.5 offset=0; type revolute -> mimic
- joint rightHipPitchKneeFrontBracket_to_rightKneeSecondaryHangar: mimic (none) -> joint=rightHipPitchKneeMotors_to_rightHipPitchKneeFrontBracket multiplier=-2.5 offset=0; type revolute -> mimic
- joint rightHipPitchKneeMotors_to_rightHipPitchKneeRearBracket: mimic joint=rightHipPitchKneeMotors_to_rightHipPitchKneeFrontBracket multiplier=0.5 offset=0 -> joint=rightHipPitchKneeMotors_to_rightHipPitchKneeFrontBracket multiplier=1.2 offset=0
- joint rightKneePrimaryHangar_to_rightCalf: mimic (none) -> joint=rightHipPitchKneeMotors_to_rightHipPitchKneeFrontBracket multiplier=-1 offset=0; type revolute -> mimic
